Commit message: Cleanup configuration files

File: drive_controller_ws/src/hw_description/urdf/husky.urdf.xacro (robot description, xacro)
@@ -22,21 +22,6 @@
 -->
 <robot name="husky" xmlns:xacro="http://ros.org/wiki/xacro">
-  <xacro:arg name="laser_enabled" default="false" />
-  <xacro:arg name="laser_xyz" default="$(optenv HUSKY_LMS1XX_XYZ 0.2206 0.0 0.00635)" />
-  <xacro:arg name="laser_rpy" default="$(optenv HUSKY_LMS1XX_RPY 0.0 0.0 0.0)" />
-  <xacro:arg name="realsense_enabled" default="false" />
-  <xacro:arg name="realsense_xyz" default="$(optenv HUSKY_REALSENSE_XYZ 0 0 0)" />
-  <xacro:arg name="realsense_rpy" default="$(optenv HUSKY_REALSENSE_RPY 0 0 0)" />
-  <xacro:arg name="realsense_mount" default="$(optenv HUSKY_REALSENSE_MOUNT_FRAME sensor_arch_mount_link)" />
-  <xacro:property name="husky_front_bumper_extend" value="$(optenv HUSKY_FRONT_BUMPER_EXTEND 0)" />
-  <xacro:property name="husky_rear_bumper_extend" value="$(optenv HUSKY_REAR_BUMPER_EXTEND 0)" />
   <xacro:arg name="robot_namespace" default="/" />
-  <!-- <xacro:arg name="urdf_extras" default="empty.urdf" /> -->
-  <!-- Included URDF/XACRO Files -->
-  <!-- <xacro:include filename="$(find husky_description)/urdf/decorations.urdf.xacro" /> -->
   <xacro:include filename="$(find hw_description)/urdf/wheel.urdf.xacro" />
-  <!-- <xacro:include filename="$(find husky_description)/urdf/accessories/intel_realsense.urdf.xacro"/>
-  <xacro:include filename="$(find husky_description)/urdf/accessories/sick_lms1xx_mount.urdf.xacro"/>
-  <xacro:include filename="$(find husky_description)/urdf/accessories/sensor_arch.urdf.xacro"/> -->
   <xacro:property name="M_PI" value="3.14159"/>
   <!-- Base Size -->
@@ -53,17 +38,4 @@
   <!-- Base link is the center of the robot's bottom plate -->
   <link name="base_link">
-    <!-- <visual>
-      <origin xyz="0 0 0" rpy="0 0 0" />
-      <geometry>
-        <mesh filename="package://husky_description/meshes/base_link.dae" />
-        <mesh filename="package://husky_description/meshes/base_link.dae" />
-      </geometry>
-    </visual> -->
-    <collision>
-      <origin xyz="${( husky_front_bumper_extend - husky_rear_bumper_extend ) / 2.0} 0 ${base_z_size/4}" rpy="0 0 0" />
-      <geometry>
-        <box size="${ base_x_size + husky_front_bumper_extend + husky_rear_bumper_extend } ${base_y_size} ${base_z_size/2}"/>
-      </geometry>
-    </collision>
     <collision>
       <origin xyz="0 0 ${base_z_size*3/4-0.01}" rpy="0 0 0" />
@@ -80,27 +52,4 @@
     <child link="base_footprint" />
   </joint>
-  <!-- Interial link stores the robot's inertial information -->
-  <link name="inertial_link">
-    <inertial>
-      <mass value="46.034" />
-      <origin xyz="-0.00065 -0.085 0.062" />
-      <inertia ixx="0.6022" ixy="-0.02364" ixz="-0.1197" iyy="1.7386" iyz="-0.001544" izz="2.0296" />
-    </inertial>
-  </link>
-  <joint name="inertial_joint" type="fixed">
-    <origin xyz="0 0 0" rpy="0 0 0" />
-    <parent link="base_link" />
-    <child link="inertial_link" />
-  </joint>
-  <!-- IMU Link is the standard mounting position for the UM6 IMU.-->
-  <!-- Can be modified with environment variables in /etc/ros/setup.bash -->
-  <link name="imu_link"/>
-  <joint name="imu_joint" type="fixed">
-    <origin xyz="$(optenv HUSKY_IMU_XYZ 0.19 0 0.149)" rpy="$(optenv HUSKY_IMU_RPY 0 -1.5708 3.1416)" />
-    <parent link="base_link" />
-    <child link="imu_link" />
-  </joint>
-  <gazebo reference="imu_link">
-  </gazebo>
   <!-- Husky wheel macros -->
   <xacro:husky_wheel wheel_prefix="front_left">
@@ -116,68 +65,3 @@
     <origin xyz="${-wheelbase/2} ${-track/2} ${wheel_vertical_offset}" rpy="0 0 0" />
   </xacro:husky_wheel>
-  <!-- <xacro:husky_decorate /> -->
-  <xacro:if value="$(arg laser_enabled)">
-    <sick_lms1xx_mount prefix="base"/>
-    <sick_lms1xx frame="base_laser" topic="scan" robot_namespace="$(arg robot_namespace)"/>
-    <joint name="laser_mount_joint" type="fixed">
-      <origin xyz="$(arg laser_xyz)" rpy="$(arg laser_rpy)" />
-      <parent link="top_plate_link" />
-      <child link="base_laser_mount" />
-    </joint>
-  </xacro:if>
-  <!-- top sensor arch; include this if we have the realsense enabled -->
-  <xacro:property name="topbar_needed_realsense" value="$(arg realsense_enabled)" />
-  <!-- In melodic we can treat the above as booleans, but in kinetic they're strings, hence this ugliness... -->
-  <xacro:if value="${topbar_needed_realsense == 'true' or topbar_needed_realsense == '1'}">
-    <xacro:sensor_arch prefix="" parent="top_plate_link">
-      <origin xyz="-0.35 0 0.51" rpy="0 0 -3.14"/>
-    </xacro:sensor_arch>
-  </xacro:if>
-  <!-- add the intel realsense to the topbar if needed -->
-  <xacro:if value="$(arg realsense_enabled)">
-    <link name="realsense_mountpoint"/>
-    <joint name="realsense_mountpoint_joint" type="fixed">
-      <origin xyz="0 0 0" rpy="0 0 -3.14159" />
-      <parent link="$(arg realsense_mount)"/>
-      <child link="realsense_mountpoint" />
-    </joint>
-    <xacro:intel_realsense_mount prefix="camera" topic="realsense" parent_link="realsense_mountpoint"/>
-  </xacro:if>
-  <gazebo>
-    <plugin name="gazebo_ros_control" filename="libgazebo_ros_control.so">
-      <robotNamespace>$(arg robot_namespace)</robotNamespace>
-      <legacyModeNS>true</legacyModeNS>
-    </plugin>
-  </gazebo>
-  <gazebo>
-    <plugin name="imu_controller" filename="libhector_gazebo_ros_imu.so">
-      <robotNamespace>$(arg robot_namespace)</robotNamespace>
-      <updateRate>50.0</updateRate>
-      <bodyName>base_link</bodyName>
-      <topicName>imu/data</topicName>
-      <accelDrift>0.005 0.005 0.005</accelDrift>
-      <accelGaussianNoise>0.005 0.005 0.005</accelGaussianNoise>
-      <rateDrift>0.005 0.005 0.005 </rateDrift>
-      <rateGaussianNoise>0.005 0.005 0.005 </rateGaussianNoise>
-      <headingDrift>0.005</headingDrift>
-      <headingGaussianNoise>0.005</headingGaussianNoise>
-    </plugin>
-  </gazebo>
-  <gazebo>
-    <plugin name="gps_controller" filename="libhector_gazebo_ros_gps.so">
-      <robotNamespace>$(arg robot_namespace)</robotNamespace>
-      <updateRate>40</updateRate>
-      <bodyName>base_link</bodyName>
-      <frameId>base_link</frameId>
-      <topicName>navsat/fix</topicName>
-      <velocityTopicName>navsat/vel</velocityTopicName>
-      <referenceLatitude>49.9</referenceLatitude>
-      <referenceLongitude>8.9</referenceLongitude>
-      <referenceHeading>0</referenceHeading>
-      <referenceAltitude>0</referenceAltitude>
-      <drift>0.0001 0.0001 0.0001</drift>
-    </plugin>
-  </gazebo>
-  <!-- Optional custom includes. -->
-  <!-- <xacro:include filename="$(arg urdf_extras)" /> -->
 </robot>

File: drive_controller_ws/src/hw_description/urdf/wheel.urdf.xacro (robot description, xacro)
@@ -24,15 +24,4 @@
 	<xacro:macro name="husky_wheel" params="wheel_prefix *joint_pose">
 		<link name="${wheel_prefix}_wheel_link">
-			<inertial>
-				<mass value="2.637" />
-				<origin xyz="0 0 0" />
-				<inertia  ixx="0.02467" ixy="0" ixz="0" iyy="0.04411" iyz="0" izz="0.02467" />
-			</inertial>
-			<!-- <visual>
-				<origin xyz="0 0 0" rpy="0 0 0" />
-				<geometry>
-					<mesh filename="package://husky_description/meshes/wheel.dae" />
-				</geometry>
-			</visual> -->
 			<collision>
 				<origin xyz="0 0 0" rpy="${M_PI/2} 0 0" />
@@ -42,11 +31,4 @@
 			</collision>
 		</link>
-		<gazebo reference="${wheel_prefix}_wheel_link">
-			<mu1 value="1.0"/>
-			<mu2 value="1.0"/>
-			<kp value="10000000.0" />
-			<kd value="1.0" />
-			<fdir1 value="1 0 0"/>
-		</gazebo>
 		<joint name="${wheel_prefix}_wheel" type="continuous">
 			<parent link="base_link"/>

Commit message: TF in Rviz

File: drive_controller_ws/src/hw_description/urdf/husky.urdf.xacro (robot description, xacro)
@@ -26,14 +26,20 @@
   <xacro:property name="M_PI" value="3.14159"/>
   <!-- Base Size -->
-  <xacro:property name="base_x_size" value="0.98740000" />
+  <!-- <xacro:property name="base_x_size" value="0.98740000" />
   <xacro:property name="base_y_size" value="0.57090000" />
-  <xacro:property name="base_z_size" value="0.24750000" />
+  <xacro:property name="base_z_size" value="0.24750000" /> -->
+  <xacro:property name="base_x_size" value="0.30700000" />
+  <xacro:property name="base_y_size" value="0.14500000" />
+  <xacro:property name="base_z_size" value="0.13000000" />
   <!-- Wheel Mounting Positions -->
+  <!-- <xacro:property name="wheelbase" value="0.5120" />
+  <xacro:property name="track" value="0.5708" />
+  <xacro:property name="wheel_vertical_offset" value="0.03282" /> -->
   <xacro:property name="wheelbase" value="0.5120" />
-  <xacro:property name="track" value="0.5708" />
-  <xacro:property name="wheel_vertical_offset" value="0.03282" />
+  <xacro:property name="track" value="0.1500" />
+  <xacro:property name="wheel_vertical_offset" value="0.00000" />
   <!-- Wheel Properties -->
-  <xacro:property name="wheel_length" value="0.1143" />
-  <xacro:property name="wheel_radius" value="0.1651" />
+  <xacro:property name="wheel_length" value="0.0400" />
+  <xacro:property name="wheel_radius" value="0.0470" />
   <!-- Base link is the center of the robot's bottom plate -->
   <link name="base_link">
@@ -53,5 +59,5 @@
   </joint>
   <!-- Husky wheel macros -->
-  <xacro:husky_wheel wheel_prefix="front_left">
+  <!-- <xacro:husky_wheel wheel_prefix="front_left">
     <origin xyz="${wheelbase/2} ${track/2} ${wheel_vertical_offset}" rpy="0 0 0" />
   </xacro:husky_wheel>
@@ -64,4 +70,10 @@
   <xacro:husky_wheel wheel_prefix="rear_right">
     <origin xyz="${-wheelbase/2} ${-track/2} ${wheel_vertical_offset}" rpy="0 0 0" />
+  </xacro:husky_wheel> -->
+  <xacro:husky_wheel wheel_prefix="left">
+    <origin xyz="0 ${track/2} 0" rpy="0 0 0" />
+  </xacro:husky_wheel>
+  <xacro:husky_wheel wheel_prefix="right">
+    <origin xyz="0 ${-track/2} 0" rpy="0 0 0" />
   </xacro:husky_wheel>
 </robot>

Commit message: Set urdf parameters

File: drive_controller_ws/src/hw_description/urdf/husky.urdf.xacro (robot description, xacro)
@@ -37,5 +37,5 @@
   <xacro:property name="wheel_vertical_offset" value="0.03282" /> -->
   <xacro:property name="wheelbase" value="0.5120" />
-  <xacro:property name="track" value="0.1500" />
+  <xacro:property name="track" value="0.1940" />
   <xacro:property name="wheel_vertical_offset" value="0.00000" />
   <!-- Wheel Properties -->
@@ -45,7 +45,8 @@
   <link name="base_link">
     <collision>
-      <origin xyz="0 0 ${base_z_size*3/4-0.01}" rpy="0 0 0" />
+      <!-- <origin xyz="0 0 ${base_z_size*3/4-0.01}" rpy="0 0 0" /> -->
+      <origin xyz="0 0 0" rpy="0 0 0" />
       <geometry>
-        <box size="${base_x_size*4/5} ${base_y_size} ${base_z_size/2-0.02}"/>
+        <box size="${base_x_size} ${base_y_size} ${base_z_size}"/>
       </geometry>
     </collision>
@@ -54,26 +55,13 @@
   <link name="base_footprint"/>
   <joint name="base_footprint_joint" type="fixed">
-    <origin xyz="0 0 ${wheel_vertical_offset - wheel_radius}" rpy="0 0 0" />
+	  <origin xyz="0 0 ${-base_z_size/2}" rpy="0 0 0" />
     <parent link="base_link" />
     <child link="base_footprint" />
   </joint>
-  <!-- Husky wheel macros -->
-  <!-- <xacro:husky_wheel wheel_prefix="front_left">
-    <origin xyz="${wheelbase/2} ${track/2} ${wheel_vertical_offset}" rpy="0 0 0" />
-  </xacro:husky_wheel>
-  <xacro:husky_wheel wheel_prefix="front_right">
-    <origin xyz="${wheelbase/2} ${-track/2} ${wheel_vertical_offset}" rpy="0 0 0" />
-  </xacro:husky_wheel>
-  <xacro:husky_wheel wheel_prefix="rear_left">
-    <origin xyz="${-wheelbase/2} ${track/2} ${wheel_vertical_offset}" rpy="0 0 0" />
-  </xacro:husky_wheel>
-  <xacro:husky_wheel wheel_prefix="rear_right">
-    <origin xyz="${-wheelbase/2} ${-track/2} ${wheel_vertical_offset}" rpy="0 0 0" />
-  </xacro:husky_wheel> -->
   <xacro:husky_wheel wheel_prefix="left">
-    <origin xyz="0 ${track/2} 0" rpy="0 0 0" />
+	  <origin xyz="0 ${track/2} ${-base_z_size/2 + wheel_radius}" rpy="0 0 0" />
   </xacro:husky_wheel>
   <xacro:husky_wheel wheel_prefix="right">
-    <origin xyz="0 ${-track/2} 0" rpy="0 0 0" />
+	  <origin xyz="0 ${-track/2} ${-base_z_size/2 + wheel_radius}" rpy="0 0 0" />
   </xacro:husky_wheel>
 </robot>

Commit message: Control parameters

File: drive_controller_ws/src/hw_description/urdf/husky.urdf.xacro (robot description, xacro)
@@ -36,10 +36,9 @@
   <xacro:property name="track" value="0.5708" />
   <xacro:property name="wheel_vertical_offset" value="0.03282" /> -->
-  <xacro:property name="wheelbase" value="0.5120" />
   <xacro:property name="track" value="0.1940" />
   <xacro:property name="wheel_vertical_offset" value="0.00000" />
   <!-- Wheel Properties -->
   <xacro:property name="wheel_length" value="0.0400" />
-  <xacro:property name="wheel_radius" value="0.0470" />
+  <xacro:property name="wheel_radius" value="0.0235" />
   <!-- Base link is the center of the robot's bottom plate -->
   <link name="base_link">
